File: apa_clockface.kicad_pcb (KiCad board)
At the start: 2 copper layers, 70 x 75 mm, 19 parts, among them J1 Conn_01x04_Female

Commit message: Finish routing, change 1x4 connector.
Parts:
- J1: footprint Connector_PinHeader_1.00mm:PinHeader_1x04_P1.00mm_Vertical -> Connector_PinHeader_2.54mm:PinHeader_1x04_P2.54mm_Vertical
- moved J1 1.41 mm to (139.0, 53.0)
Routing:
- net +5V: track 26.9 -> 80.0 mm, vias 0 -> 8
- net Net-(D1-Pad2): track 17.2 -> 21.1 mm
- net Net-(D1-Pad1): track 14.6 -> 16.7 mm
- net Net-(D7-Pad5): track 10.2 -> 12.1 mm
- net Net-(D1-Pad5): track 9.75 -> 10.6 mm
- net GND: track 2.03 -> 1.29 mm
- net (no net): vias 1 -> 0
Other:
- rule trace_min: 0.2 -> 0.08
- rule via_min_size: 0.4 -> 0.2
